Commit message: trying to add controller

File: urdf/robot_arm.urdf (robot description, URDF)
Before this commit: robot robot_arm, 7 links, 6 joints
Links:
- added link body0, mass 0.341; visual box size=0.15 0.02 0.02
- added link body1, mass 0.194; visual box size=0.02 0.02 0.05
- added link body2, mass 0.429; visual box size=0.15 0.02 0.02
- added link body3, mass 0.115; visual box size=0.02 0.02 0.02
- added link body4, mass 0.333; visual box size=0.02 0.02 0.16
- link link1: mass 0.194 -> None; geometry visual cylinder length=0.04 radius=0.015
- link link2: mass 0.194 -> None; geometry visual cylinder length=0.04 radius=0.015
- link link3: mass 0.194 -> None; geometry visual cylinder length=0.04 radius=0.015
- link link4: mass 0.194 -> None; geometry visual box size=0.01 0.01 0.01
- link link5: mass 0.194 -> None; geometry visual box size=0.01 0.01 0.01
Joints:
- added joint base_link_to_body0: type fixed, parent base_link, child body0, origin xyz=0 0 0 rpy=0 0 0
- added joint link0_to_body1: type fixed, parent link0, child body1, origin xyz=0 0 0 rpy=0 0 0
- added joint link1_to_body2: type fixed, parent link1, child body2, origin xyz=0 0 0 rpy=0 0 0
- added joint link2_to_body3: type fixed, parent link2, child body3, origin xyz=0 0 0 rpy=0 0 0
- added joint link3_to_body4: type fixed, parent link3, child body4, origin xyz=0 0 0 rpy=0 0 0

File: xacro/link0.xacro (robot description, xacro)
@@ -2,4 +2,23 @@
 <robot xmlns:xacro="http://www.ros.org/wiki/xacro">
   <xacro:macro name="link0" params="parent">
+    <link name="body0">
+      <visual>
+        <origin xyz="-0.075 0 0" rpy="0 0 0" />
+        <geometry>
+          <box size="0.15 0.02 0.02"/>
+        </geometry>
+        <material name="grey"/>
+      </visual>
+      <inertial>
+        <mass value="0.341"/>
+        <origin xyz="-0.075 -0.006 -0.003"/>
+        <inertia ixx="0.000099" ixy="0.000139" ixz="0.000115" iyy="0.002920" iyz="0.000003" izz="0.002934"/>
+      </inertial>
+    </link>
+    <joint name="base_link_to_body0" type="fixed">
+      <origin xyz="0 0 0" rpy="0 0 0"/>
+      <parent link="${parent}"/>
+      <child link="body0"/>
+    </joint>
     <link name="link0">
       <visual>
@@ -7,9 +26,9 @@
           <cylinder radius="0.015" length="0.04"/>
         </geometry>
-        <origin xyz="0 0 0" rpy="0 0 0"/>
       </visual>
     </link>
     <joint name="joint1" type="revolute">
       <axis xyz="0 0 1"/>
+      <dynamics damping="1.0" friction="1.0"/>
       <limit effort="1" lower="-3.1416" upper="3.1416" velocity="0.5"/>
       <origin xyz="0 0 0" rpy="0 0 0"/>

File: xacro/link1.xacro (robot description, xacro)
@@ -2,4 +2,23 @@
 <robot xmlns:xacro="http://www.ros.org/wiki/xacro">
   <xacro:macro name="link1" params="parent">
+    <link name="body1">
+      <visual>
+        <origin xyz="0 0 0.02" rpy="0 0 0" />
+        <geometry>
+          <box size="0.02 0.02 0.05"/>
+        </geometry>
+        <material name="grey"/>
+      </visual>
+      <inertial>
+        <mass value="0.194"/>
+        <origin xyz="0.005 -0.001 0.016"/>
+        <inertia ixx="0.000189" ixy="0.000005" ixz="0.000054" iyy="0.000213" iyz="0.000003" izz="0.000067"/>
+      </inertial>
+    </link>
+    <joint name="link0_to_body1" type="fixed">
+      <origin xyz="0 0 0" rpy="0 0 0"/>
+      <parent link="${parent}"/>
+      <child link="body1"/>
+    </joint>
     <link name="link1">
       <visual>
@@ -8,17 +27,8 @@
         </geometry>
       </visual>
-      <collision>
-        <geometry>
-          <cylinder radius="0.015" length="0.04"/>
-        </geometry>
-      </collision>
-      <inertial>
-        <mass value="0.194"/>
-        <origin xyz="0 0 0"/>
-        <inertia ixx="0.0" ixy="0.0" ixz="0.0" iyy="0.0" iyz="0.0" izz="0.0"/>
-      </inertial>
     </link>
     <joint name="joint2" type="revolute">
       <axis xyz="0 0 1"/>
+      <dynamics damping="1.0" friction="1.0"/>
       <limit effort="1" lower="-3.1416" upper="3.1416" velocity="0.5"/>
       <origin xyz="-0.02 0 0.0462" rpy="1.5707 0 3.1415"/>

File: xacro/link2.xacro (robot description, xacro)
@@ -2,4 +2,23 @@
 <robot xmlns:xacro="http://www.ros.org/wiki/xacro">
   <xacro:macro name="link2" params="parent">
+    <link name="body2">
+      <visual>
+        <origin xyz="0.075 0 0" rpy="0 0 0" />
+        <geometry>
+          <box size="0.15 0.02 0.02"/>
+        </geometry>
+        <material name="grey"/>
+      </visual>
+      <inertial>
+        <mass value="0.429"/>
+        <origin xyz="0.073 0 0"/>
+        <inertia ixx="0.000087" ixy="-0.000076" ixz="-0.000010" iyy="0.003190" iyz="0" izz="0.003213"/>
+      </inertial>
+    </link>
+    <joint name="link1_to_body2" type="fixed">
+      <origin xyz="0 0 0" rpy="0 0 0"/>
+      <parent link="${parent}"/>
+      <child link="body2"/>
+    </joint>
     <link name="link2">
       <visual>
@@ -8,17 +27,8 @@
         </geometry>
       </visual>
-      <collision>
-        <geometry>
-          <cylinder radius="0.015" length="0.04"/>
-        </geometry>
-      </collision>
-      <inertial>
-        <mass value="0.194"/>
-        <origin xyz="0 0 0"/>
-        <inertia ixx="0.0" ixy="0.0" ixz="0.0" iyy="0.0" iyz="0.0" izz="0.0"/>
-      </inertial>
     </link>
     <joint name="joint3" type="revolute">
       <axis xyz="0 0 1"/>
+      <dynamics damping="1.0" friction="1.0"/>
       <limit effort="1" lower="-3.1416" upper="3.1416" velocity="0.5"/>
       <origin xyz="0.15071 0 0" rpy="3.1415 0 0"/>

File: xacro/link3.xacro (robot description, xacro)
@@ -2,4 +2,23 @@
 <robot xmlns:xacro="http://www.ros.org/wiki/xacro">
   <xacro:macro name="link3" params="parent">
+    <link name="body3">
+      <visual>
+        <origin xyz="0 -0.02 0" rpy="0 0 0" />
+        <geometry>
+          <box size="0.02 0.02 0.02"/>
+        </geometry>
+        <material name="grey"/>
+      </visual>
+      <inertial>
+        <mass value="0.115"/>
+        <origin xyz="0.017 -0.026 -0.002"/>
+        <inertia ixx="0.000120" ixy="-0.000061" ixz="-0.000001" iyy="0.000062" iyz="0" izz="0.000156"/>
+      </inertial>
+    </link>
+    <joint name="link2_to_body3" type="fixed">
+      <origin xyz="0 0 0" rpy="0 0 0"/>
+      <parent link="${parent}"/>
+      <child link="body3"/>
+    </joint>
     <link name="link3">
       <visual>
@@ -8,17 +27,8 @@
         </geometry>
       </visual>
-      <collision>
-        <geometry>
-          <cylinder radius="0.015" length="0.04"/>
-        </geometry>
-      </collision>
-      <inertial>
-        <mass value="0.194"/>
-        <origin xyz="0 0 0"/>
-        <inertia ixx="0.0" ixy="0.0" ixz="0.0" iyy="0.0" iyz="0.0" izz="0.0"/>
-      </inertial>
     </link>
     <joint name="joint4" type="revolute">
       <axis xyz="0 0 1"/>
+      <dynamics damping="1.0" friction="1.0"/>
       <limit effort="1" lower="-3.1416" upper="3.1416" velocity="0.5"/>
       <origin xyz="0.00531 -0.01928 0" rpy=" -1.5707 0 -1.3021"/>

File: xacro/link4.xacro (robot description, xacro)
@@ -2,4 +2,23 @@
 <robot xmlns:xacro="http://www.ros.org/wiki/xacro">
   <xacro:macro name="link4" params="parent">
+    <link name="body4">
+      <visual>
+        <origin xyz="0 0 -0.08" rpy="0 0 0" />
+        <geometry>
+          <box size="0.02 0.02 0.16"/>
+        </geometry>
+        <material name="grey"/>
+      </visual>
+      <inertial>
+        <mass value="0.333"/>
+        <origin xyz="0 0.003 -0.098"/>
+        <inertia ixx="0.003709" ixy="0.000002" ixz="-0.000004" iyy="0.003734" iyz="0" izz="0.000079"/>
+      </inertial>
+    </link>
+    <joint name="link3_to_body4" type="fixed">
+      <origin xyz="0 0 0" rpy="0 0 0"/>
+      <parent link="${parent}"/>
+      <child link="body4"/>
+    </joint>
     <link name="link4">
       <visual>
@@ -8,14 +27,4 @@
         </geometry>
       </visual>
-      <collision>
-        <geometry>
-          <box size="0.01 0.01 0.01"/>
-        </geometry>
-      </collision>
-      <inertial>
-        <mass value="0.194"/>
-        <origin xyz="0 0 0"/>
-        <inertia ixx="0.0" ixy="0.0" ixz="0.0" iyy="0.0" iyz="0.0" izz="0.0"/>
-      </inertial>
     </link>
     <joint name="link3_to_link4" type="fixed">

File: xacro/link5.xacro (robot description, xacro)
@@ -8,14 +8,4 @@
         </geometry>
       </visual>
-      <collision>
-        <geometry>
-          <box size="0.01 0.01 0.01"/>
-        </geometry>
-      </collision>
-      <inertial>
-        <mass value="0.194"/>
-        <origin xyz="0 0 0"/>
-        <inertia ixx="0.0" ixy="0.0" ixz="0.0" iyy="0.0" iyz="0.0" izz="0.0"/>
-      </inertial>
     </link>
     <joint name="link4_to_link5" type="fixed">

File: xacro/main.xacro (robot description, xacro)
@@ -3,4 +3,5 @@
     <link name="base_link"></link>
     <!-- Include the Modular Xacro Files -->
+    <xacro:include filename="include.xacro"/>
     <xacro:include filename="link0.xacro"/>
     <xacro:include filename="link1.xacro"/>
@@ -9,4 +10,5 @@
     <xacro:include filename="link4.xacro"/>
     <xacro:include filename="link5.xacro"/>
+    <!-- <xacro:include filename="plugins.xacro"/> -->
     <xacro:link0 parent="base_link"/>
     <xacro:link1 parent="link0"/>

Commit message: ble

File: urdf/robot_arm.urdf (robot description, URDF)
Before this commit: robot robot_arm, 12 links, 11 joints
Joints:
- joint joint1: limit lower=-3.1416 upper=3.1416 effort=1 velocity=0.5 -> lower=-3.1416 upper=3.1416 effort=100 velocity=0.5
- joint joint2: limit lower=-3.1416 upper=3.1416 effort=1 velocity=0.5 -> lower=-3.1416 upper=3.1416 effort=100 velocity=0.5
- joint joint3: limit lower=-3.1416 upper=3.1416 effort=1 velocity=0.5 -> lower=-3.1416 upper=3.1416 effort=100 velocity=0.5
- joint joint4: limit lower=-3.1416 upper=3.1416 effort=1 velocity=0.5 -> lower=-3.1416 upper=3.1416 effort=100 velocity=0.5

File: xacro/link0.xacro (robot description, xacro)
@@ -31,9 +31,15 @@
       <axis xyz="0 0 1"/>
       <dynamics damping="1.0" friction="1.0"/>
-      <limit effort="1" lower="-3.1416" upper="3.1416" velocity="0.5"/>
+      <limit effort="100" lower="-3.1416" upper="3.1416" velocity="0.5"/>
       <origin xyz="0 0 0" rpy="0 0 0"/>
       <parent link="${parent}"/>
       <child link="link0"/>
     </joint>
+    <transmission name="joint1_transmission">
+      <type>transmission_interface/SimpleTransmission</type>
+      <joint name="joint1">
+        <hardwareInterface>hardware_interface/PositionJointInterface</hardwareInterface>
+      </joint>
+    </transmission>
   </xacro:macro>
 </robot>

File: xacro/link1.xacro (robot description, xacro)
@@ -31,9 +31,15 @@
       <axis xyz="0 0 1"/>
       <dynamics damping="1.0" friction="1.0"/>
-      <limit effort="1" lower="-3.1416" upper="3.1416" velocity="0.5"/>
+      <limit effort="100" lower="-3.1416" upper="3.1416" velocity="0.5"/>
       <origin xyz="-0.02 0 0.0462" rpy="1.5707 0 3.1415"/>
       <parent link="${parent}"/>
       <child link="link1"/>
     </joint>
+    <transmission name="joint2_transmission">
+      <type>transmission_interface/SimpleTransmission</type>
+      <joint name="joint2">
+        <hardwareInterface>hardware_interface/PositionJointInterface</hardwareInterface>
+      </joint>
+    </transmission>
   </xacro:macro>
 </robot>

File: xacro/link2.xacro (robot description, xacro)
@@ -31,9 +31,15 @@
       <axis xyz="0 0 1"/>
       <dynamics damping="1.0" friction="1.0"/>
-      <limit effort="1" lower="-3.1416" upper="3.1416" velocity="0.5"/>
+      <limit effort="100" lower="-3.1416" upper="3.1416" velocity="0.5"/>
       <origin xyz="0.15071 0 0" rpy="3.1415 0 0"/>
       <parent link="${parent}"/>
       <child link="link2"/>
     </joint>
+    <transmission name="joint3_transmission">
+      <type>transmission_interface/SimpleTransmission</type>
+      <joint name="joint3">
+        <hardwareInterface>hardware_interface/PositionJointInterface</hardwareInterface>
+      </joint>
+    </transmission>
   </xacro:macro>
 </robot>

File: xacro/link3.xacro (robot description, xacro)
@@ -31,9 +31,15 @@
       <axis xyz="0 0 1"/>
       <dynamics damping="1.0" friction="1.0"/>
-      <limit effort="1" lower="-3.1416" upper="3.1416" velocity="0.5"/>
+      <limit effort="100" lower="-3.1416" upper="3.1416" velocity="0.5"/>
       <origin xyz="0.00531 -0.01928 0" rpy=" -1.5707 0 -1.3021"/>
       <parent link="${parent}"/>
       <child link="link3"/>
     </joint>
+    <transmission name="joint4_transmission">
+      <type>transmission_interface/SimpleTransmission</type>
+      <joint name="joint4">
+        <hardwareInterface>hardware_interface/PositionJointInterface</hardwareInterface>
+      </joint>
+    </transmission>
   </xacro:macro>
 </robot>
